Commit message: add hedge adaptor and launch file

File: ws/src/drift_sim/urdf/drift_car.urdf.xacro (robot description, xacro)
@@ -36,5 +36,5 @@
        along the y axis, and chassis_height along the z axis. -->
   <xacro:property name="chassis_length" value="0.32"/>
-  <xacro:property name="chassis_width" value="0.09"/>
+  <xacro:property name="chassis_width" value="0.13"/>
   <xacro:property name="chassis_height" value="0.01"/>
   <xacro:property name="chassis_mass" value="2"/>
@@ -45,5 +45,5 @@
        axle_length. -->
   <xacro:property name="hub_dia" value="0.05"/>
-  <xacro:property name="tire_dia" value="0.065"/>
+  <xacro:property name="tire_dia" value="0.06"/>
   <xacro:property name="tire_width" value="0.025"/>
   <xacro:property name="hex_hub_depth" value="0.012"/>
@@ -54,7 +54,7 @@
        vertical wheel travel. -->
   <xacro:property name="wheelbase" value="0.26"/>
-  <xacro:property name="hex_hub_dist" value="0.23"/>
+  <xacro:property name="hex_hub_dist" value="0.17"/>
   <xacro:property name="axle_length" value="0.01"/>
-  <xacro:property name="wheel_travel" value="0.01"/>
+  <xacro:property name="wheel_travel" value="0.015"/>
   <xacro:property name="shock_z_offset" value="0.0655"/>
   <!-- The specifications for a Titan(R) 550 motor could not be found, so the
@@ -238,7 +238,32 @@
     <material>Gazebo/Red</material>
   </gazebo>
+  <joint name="hedge_joint" type="fixed">
+		<axis xyz="1 0 0"/>
+		<origin xyz="-0.16 0.0 0.08"/>
+		<parent link="base_link"/>
+		<child link="hedge_link"/>
+  </joint>
+	<link name="hedge_link">
+	  <inertial>
+	    <mass value="0.001"/>
+	    <origin rpy="0 0 0" xyz="0 0 0"/>
+	    <inertia ixx="0.0001" ixy="0" ixz="0" iyy="0.000001" iyz="0" izz="0.0001"/>
+	  </inertial>
+	  <visual>
+	    <origin rpy="0 0 0" xyz="0 0 0"/>
+	    <geometry>
+	      <box size="0.001 0.001 0.001"/>
+	    </geometry>
+	  </visual>
+	  <collision>
+	    <origin rpy="0 0 0" xyz="0 0 0"/>
+	    <geometry>
+	      <box size=".001 .001 .001"/>
+	    </geometry>
+	  </collision>
+	</link>
   <joint name="imu_joint" type="fixed">
 		<axis xyz="1 0 0"/>
-		<origin xyz="0 0 0.19"/>
+		<origin xyz="-0.16 0.025 0.19"/>
 		<parent link="base_link"/>
 		<child link="imu_link"/>

Commit message: working rc car env and tuned params

File: ws/src/drift_sim/urdf/drift_car.urdf.xacro (robot description, xacro)
@@ -30,4 +30,5 @@
   <!-- Degree-to-radian conversions -->
   <xacro:property name="degrees_15" value="0.261799"/>
+  <xacro:property name="degrees_21" value="0.366519"/>
   <xacro:property name="degrees_25" value="0.436332"/>
   <xacro:property name="degrees_45" value="0.785398163"/>
@@ -38,5 +39,5 @@
   <xacro:property name="chassis_width" value="0.13"/>
   <xacro:property name="chassis_height" value="0.01"/>
-  <xacro:property name="chassis_mass" value="2"/>
+  <xacro:property name="chassis_mass" value="2.5"/>
   <!-- hub_dia and tire_dia are the diameters of the hub and tire,
        respectively. hex_hub_depth is the distance that the hex hub is
@@ -200,5 +201,5 @@
       <child link="${lr_prefix}_${fr_prefix}_axle_carrier"/>
       <axis xyz="0 0 1"/>
-      <limit lower="${-degrees_45}" upper="${degrees_45}"
+      <limit lower="${-degrees_21}" upper="${degrees_21}"
              effort="${servo_stall_torque}" velocity="${servo_no_load_speed}"/>
     </joint>
@@ -214,5 +215,5 @@
     </transmission>
     <xacro:wheel lr_prefix="${lr_prefix}" fr_prefix="${fr_prefix}"
-                 lr_reflect="${lr_reflect}" mu1="0.5" mu2="0.5"/>
+                 lr_reflect="${lr_reflect}" mu1="0.3" mu2="0.3"/>
   </xacro:macro>
   <!-- Rear wheel -->
@@ -223,5 +224,5 @@
                  child="${lr_prefix}_${fr_prefix}_axle_carrier"/>
     <xacro:wheel lr_prefix="${lr_prefix}" fr_prefix="${fr_prefix}"
-                 lr_reflect="${lr_reflect}" mu1="0.5" mu2="0.5"/>
+                 lr_reflect="${lr_reflect}" mu1="0.3" mu2="0.3"/>
   </xacro:macro>
   <!-- base_link must have geometry so that its axes can be displayed in

Commit message: more parameter updates

File: ws/src/drift_sim/urdf/drift_car.urdf.xacro (robot description, xacro)
@@ -39,5 +39,5 @@
   <xacro:property name="chassis_width" value="0.13"/>
   <xacro:property name="chassis_height" value="0.01"/>
-  <xacro:property name="chassis_mass" value="2.5"/>
+  <xacro:property name="chassis_mass" value="15.0"/>
   <!-- hub_dia and tire_dia are the diameters of the hub and tire,
        respectively. hex_hub_depth is the distance that the hex hub is
@@ -49,5 +49,5 @@
   <xacro:property name="tire_width" value="0.025"/>
   <xacro:property name="hex_hub_depth" value="0.012"/>
-  <xacro:property name="wheel_mass" value="0.3"/>
+  <xacro:property name="wheel_mass" value="0.18"/>
   <!-- hex_hub_dist is the distance between left and right hex hubs when
        the shock absorbers are fully extended. axle_length is the distance
@@ -71,5 +71,7 @@
        axle_vel_limit = (2 * pi) * (max_speed / (pi * tire_dia)) =
          550.203076923 rad/s -->
-  <xacro:property name="axle_eff_limit" value="4.388225625"/>
+  <!-- <xacro:property name="axle_eff_limit" value="4.388225625"/> -->
+  <xacro:property name="axle_eff_limit" value="2.888225625"/>
+  <!-- <xacro:property name="axle_vel_limit" value="550.203076923"/> -->
   <xacro:property name="axle_vel_limit" value="550.203076923"/>
   <!-- These constants are used to simulate a Traxxas 2056 servo operated at
@@ -215,5 +217,5 @@
     </transmission>
     <xacro:wheel lr_prefix="${lr_prefix}" fr_prefix="${fr_prefix}"
-                 lr_reflect="${lr_reflect}" mu1="0.3" mu2="0.3"/>
+                 lr_reflect="${lr_reflect}" mu1="0.40" mu2="0.40"/>
   </xacro:macro>
   <!-- Rear wheel -->
@@ -224,5 +226,5 @@
                  child="${lr_prefix}_${fr_prefix}_axle_carrier"/>
     <xacro:wheel lr_prefix="${lr_prefix}" fr_prefix="${fr_prefix}"
-                 lr_reflect="${lr_reflect}" mu1="0.3" mu2="0.3"/>
+                 lr_reflect="${lr_reflect}" mu1="0.40" mu2="0.40"/>
   </xacro:macro>
   <!-- base_link must have geometry so that its axes can be displayed in

Commit message: add pilco python implementation

File: ws/src/drift_sim/urdf/drift_car.urdf.xacro (robot description, xacro)
@@ -39,5 +39,5 @@
   <xacro:property name="chassis_width" value="0.13"/>
   <xacro:property name="chassis_height" value="0.01"/>
-  <xacro:property name="chassis_mass" value="15.0"/>
+  <xacro:property name="chassis_mass" value="8.0"/>
   <!-- hub_dia and tire_dia are the diameters of the hub and tire,
        respectively. hex_hub_depth is the distance that the hex hub is
@@ -49,5 +49,5 @@
   <xacro:property name="tire_width" value="0.025"/>
   <xacro:property name="hex_hub_depth" value="0.012"/>
-  <xacro:property name="wheel_mass" value="0.18"/>
+  <xacro:property name="wheel_mass" value="0.20"/>
   <!-- hex_hub_dist is the distance between left and right hex hubs when
        the shock absorbers are fully extended. axle_length is the distance
@@ -203,5 +203,5 @@
       <child link="${lr_prefix}_${fr_prefix}_axle_carrier"/>
       <axis xyz="0 0 1"/>
-      <limit lower="${-degrees_21}" upper="${degrees_21}"
+      <limit lower="${-degrees_45}" upper="${degrees_45}"
              effort="${servo_stall_torque}" velocity="${servo_no_load_speed}"/>
     </joint>
@@ -217,5 +217,5 @@
     </transmission>
     <xacro:wheel lr_prefix="${lr_prefix}" fr_prefix="${fr_prefix}"
-                 lr_reflect="${lr_reflect}" mu1="0.40" mu2="0.40"/>
+                 lr_reflect="${lr_reflect}" mu1="0.45" mu2="0.45"/>
   </xacro:macro>
   <!-- Rear wheel -->
@@ -226,5 +226,5 @@
                  child="${lr_prefix}_${fr_prefix}_axle_carrier"/>
     <xacro:wheel lr_prefix="${lr_prefix}" fr_prefix="${fr_prefix}"
-                 lr_reflect="${lr_reflect}" mu1="0.40" mu2="0.40"/>
+                 lr_reflect="${lr_reflect}" mu1="0.45" mu2="0.45"/>
   </xacro:macro>
   <!-- base_link must have geometry so that its axes can be displayed in

Commit message: new imu pos

File: ws/src/drift_sim/urdf/drift_car.urdf.xacro (robot description, xacro)
@@ -243,5 +243,5 @@
   <joint name="hedge_joint" type="fixed">
 		<axis xyz="1 0 0"/>
-		<origin xyz="-0.16 0.0 0.08"/>
+		<origin xyz="0.16 0.0 0.08"/>
 		<parent link="base_link"/>
 		<child link="hedge_link"/>
@@ -268,5 +268,5 @@
   <joint name="imu_joint" type="fixed">
 		<axis xyz="1 0 0"/>
-		<origin xyz="-0.16 0.025 0.19"/>
+		<origin xyz="0.16 0.025 0.08"/>
 		<parent link="base_link"/>
 		<child link="imu_link"/>
@@ -275,5 +275,5 @@
 	  <inertial>
 	    <mass value="0.001"/>
-	    <origin rpy="0 0 0" xyz="0 0 0"/>
+	    <origin rpy="0 0 -${degrees_90}" xyz="0 0 0"/>
 	    <inertia ixx="0.0001" ixy="0" ixz="0" iyy="0.000001" iyz="0" izz="0.0001"/>
 	  </inertial>

Commit message: imu changes

File: ws/src/drift_sim/urdf/drift_car.urdf.xacro (robot description, xacro)
@@ -275,5 +275,5 @@
 	  <inertial>
 	    <mass value="0.001"/>
-	    <origin rpy="0 0 -${degrees_90}" xyz="0 0 0"/>
+	    <origin rpy="0 0 0" xyz="0 0 0"/>
 	    <inertia ixx="0.0001" ixy="0" ixz="0" iyy="0.000001" iyz="0" izz="0.0001"/>
 	  </inertial>

Commit message: more imu changes

File: ws/src/drift_sim/urdf/drift_car.urdf.xacro (robot description, xacro)
@@ -268,5 +268,5 @@
   <joint name="imu_joint" type="fixed">
 		<axis xyz="1 0 0"/>
-		<origin xyz="0.16 0.025 0.08"/>
+		<origin xyz="0.16 0.025 0.08" rpy="0 0 -{degrees_90}"/>
 		<parent link="base_link"/>
 		<child link="imu_link"/>

Commit message: imu changes

File: ws/src/drift_sim/urdf/drift_car.urdf.xacro (robot description, xacro)
@@ -268,5 +268,5 @@
   <joint name="imu_joint" type="fixed">
 		<axis xyz="1 0 0"/>
-		<origin xyz="0.16 0.025 0.08" rpy="0 0 -{degrees_90}"/>
+		<origin xyz="0.16 0.025 0.08" rpy="0 0 -${degrees_90}"/>
 		<parent link="base_link"/>
 		<child link="imu_link"/>

Commit message: change  imu pos

File: ws/src/drift_sim/urdf/drift_car.urdf.xacro (robot description, xacro)
@@ -268,5 +268,5 @@
   <joint name="imu_joint" type="fixed">
 		<axis xyz="1 0 0"/>
-		<origin xyz="0.16 0.025 0.08" rpy="0 0 -${degrees_90}"/>
+		<origin xyz="0.16 0.025 0.08" rpy="0 0 0"/>
 		<parent link="base_link"/>
 		<child link="imu_link"/>

Commit message: change  imu pos

File: ws/src/drift_sim/urdf/drift_car.urdf.xacro (robot description, xacro)
@@ -268,5 +268,5 @@
   <joint name="imu_joint" type="fixed">
 		<axis xyz="1 0 0"/>
-		<origin xyz="0.16 0.025 0.08" rpy="0 0 0"/>
+		<origin xyz="0.16 0.025 0.08" rpy="0 0 -${degrees_90}"/>
 		<parent link="base_link"/>
 		<child link="imu_link"/>
